File: PCB V3/SLSS PCB V3/SLSS PCB V3.kicad_sch (KiCad schematic)
At the start: 0 parts

Commit message: Updated KiCad Schematic
Included arduino nano trace and USB-C connector
Parts:
- added A1: Arduino_Nano_Every_Socket, PCM_arduino-library:Arduino_Nano_Every_Socket, symbol PCM_arduino-library:Arduino_Nano_Every_Socket
- added P1: USB_C_Plug-Connector, Connector_USB:USB_C_Receptacle_Amphenol_12401548E4-2A, symbol USB-C-USB-3.2-rescue:USB_C_Plug-Connector
Connections:
- new net GND: P1.A1 (GND), P1.A12 (GND), P1.B1 (GND), P1.B12 (GND)
- new net VBUS: P1.A4 (VBUS), P1.A9 (VBUS), P1.B4 (VBUS), P1.B9 (VBUS)
Changed lines of the file:
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@@
 	(generator_version "9.0")
 	(paper "A4")
+	(symbol
+		(lib_id "PCM_arduino-library:Arduino_Nano_Every_Socket")
+		(at 142.24 71.12 0)
+		(unit 1)
+		(exclude_from_sim no)
+		(in_bom yes)
+		(on_board yes)
+		(dnp no)
+		(fields_autoplaced yes)
+		(property "Reference" "A1"
+			(at 142.24 39.37 0)
+			(effects
+				(font
+					(size 1.524 1.524)
+				)
+			)
+		)
+		(property "Value" "Arduino_Nano_Every_Socket"
+			(at 142.24 41.91 0)
+			(effects
+				(font
+					(size 1.524 1.524)
+				)
+			)
+		)
+		(property "Footprint" "PCM_arduino-library:Arduino_Nano_Every_Socket"
+			(at 142.24 105.41 0)
+			(effects
+				(font
+					(size 1.524 1.524)
+				)
+				(hide yes)
+			)
+		)
+		(property "Datasheet" "https://docs.arduino.cc/hardware/nano-every"
+			(at 142.24 101.6 0)
+			(effects
+				(font
+					(size 1.524 1.524)
+				)
+				(hide yes)
+			)
+		)
+		(property "Description" "Socket for Arduino Nano Every"
+			(at 142.24 71.12 0)
+			(effects
+				(font
+					(size 1.27 1.27)
+				)
+				(hide yes)
+			)
+		)
+		(pin "D0"
+		)
+		(pin "3V3"
+		)
+		(pin "D2"
+		)
+		(pin "GND1"
+		)
+		(pin "AREF"
+		)
+		(pin "D3"
+		)
+		(pin "A6"
+		)
+		(pin "VIN"
+		)
+		(pin "A5"
+		)
+		(pin "A1"
+		)
+		(pin "D1"
+		)
+		(pin "A7"
+		)
+		(pin "A3"
+		)
+		(pin "A4"
+		)
+		(pin "A2"
+		)
+		(pin "A0"
+		)
+		(pin "5V"
+		)
+		(pin "GND2"
+		)
+		(pin "D5"
+		)
+		(pin "D13"
+		)
+		(pin "D9"
+		)
+		(pin "D12"
+		)
+		(pin "D6"
+		)
+		(pin "D8"
+		)
+		(pin "D10"
+		)
+		(pin "D11"
+		)
+		(pin "D4"
+		)
+		(pin "RST2"
+		)
+		(pin "RST1"
+		)
+		(pin "D7"
+		)
+		(instances
+			(project ""
+				(path "/47896011-57f9-4105-b464-bed95da27d40"
+					(reference "A1")
+					(unit 1)
+				)
+			)
+		)
+	)
+	(symbol
+		(lib_id "USB-C-USB-3.2-rescue:USB_C_Plug-Connector")
+		(at 26.67 48.26 0)
+		(unit 1)
+		(exclude_from_sim no)
+		(in_bom yes)
+		(on_board yes)
+		(dnp no)
+		(fields_autoplaced yes)
+		(property "Reference" "P1"
+			(at 26.67 15.24 0)
+			(effects
+				(font
+					(size 1.27 1.27)
+				)
+			)
+		)
+		(property "Value" "USB_C_Plug-Connector"
+			(at 26.67 17.78 0)
+			(effects
+				(font
+					(size 1.27 1.27)
+				)
+			)
+		)
+		(property "Footprint" "Connector_USB:USB_C_Receptacle_Amphenol_12401548E4-2A"
+			(at 30.48 48.26 0)
+			(effects
+				(font
+					(size 1.27 1.27)
+				)
+				(hide yes)
+			)
+		)
+		(property "Datasheet" ""
+			(at 30.48 48.26 0)
+			(effects
+				(font
+					(size 1.27 1.27)
+				)
+				(hide yes)
+			)
+		)
+		(property "Description" ""
+			(at 26.67 48.26 0)
+			(effects
+				(font
+					(size 1.27 1.27)
+				)
+				(hide yes)
+			)
+		)
+		(pin "A6"
+		)
+		(pin "A4"
+		)
+		(pin "B1"
+		)
+		(pin "B8"
+		)
+		(pin "B2"
+		)
+		(pin "S1"
+		)
+		(pin "A8"
+		)
+		(pin "A2"
+		)
+		(pin "A10"
+		)
+		(pin "A1"
+		)
+		(pin "B12"
+		)
+		(pin "B11"
+		)
+		(pin "A12"
+		)
+		(pin "B5"
+		)
+		(pin "B3"
+		)
+		(pin "A5"
+		)
+		(pin "B4"
+		)
+		(pin "B9"
+		)
+		(pin "A7"
+		)
+		(pin "A9"
+		)
+		(pin "B10"
+		)
+		(pin "A11"
+		)
+		(pin "A3"
+		)
+		(instances
+			(project ""
+				(path "/47896011-57f9-4105-b464-bed95da27d40"
+					(reference "P1")
+					(unit 1)
+				)
+			)
+		)
+	)
 	(sheet_instances
 		(path "/"

Commit message: Screen documentation
Parts:
- added J1: Adafruit Screen, symbol Connector_Generic:Conn_01x04
Changed lines of the file:
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@@
+		)
+	)
+	(symbol
+		(lib_id "Connector_Generic:Conn_01x04")
+		(at 53.34 128.27 0)
+		(mirror y)
+		(unit 1)
+		(exclude_from_sim no)
+		(in_bom yes)
+		(on_board yes)
+		(dnp no)
+		(property "Reference" "J1"
+			(at 50.8 128.2699 0)
+			(effects
+				(font
+					(size 1.27 1.27)
+				)
+				(justify left)
+			)
+		)
+		(property "Value" "Adafruit Screen"
+			(at 50.8 130.8099 0)
+			(effects
+				(font
+					(size 1.27 1.27)
+				)
+				(justify left)
+			)
+		)
+		(property "Footprint" ""
+			(at 53.34 128.27 0)
+			(effects
+				(font
+					(size 1.27 1.27)
+				)
+				(hide yes)
+			)
+		)
+		(property "Datasheet" "~"
+			(at 53.34 128.27 0)
+			(effects
+				(font
+					(size 1.27 1.27)
+				)
+				(hide yes)
+			)
+		)
+		(property "Description" "Generic connector, single row, 01x04, script generated (kicad-library-utils/schlib/autogen/connector/)"
+			(at 53.34 128.27 0)
+			(effects
+				(font
+					(size 1.27 1.27)
+				)
+				(hide yes)
+			)
+		)
+		(pin "1"
+		)
+		(pin "2"
+		)
+		(pin "4"
+		)
+		(pin "3"
+		)
+		(instances
+			(project ""
+				(path "/47896011-57f9-4105-b464-bed95da27d40"
+					(reference "J1")
+					(unit 1)
+				)
+			)
 		)
 	)
